Commit message: twidling with kin plugings

File: src/gzrcs/config/lrmate200id-save.urdf (robot description, URDF)
Before this commit: robot fanuc_lrmate200id, 7 links, 6 joints
Links:
- added link base
- link fanuc_base_link: mass 4 -> None
- link fanuc_link_1: mass 4 -> None
- link fanuc_link_2: mass 5 -> None
- link fanuc_link_3: mass 4 -> None
- link fanuc_link_4: mass 5 -> None
- link fanuc_link_5: mass 1.5 -> None
- link fanuc_link_6: mass 0.25 -> None
Joints:
- added joint base_link-base: type fixed, parent fanuc_base_link, child base, origin xyz=0 0 0 rpy=0 0 0
- joint fanuc_joint_1: origin xyz=0 0 0.33 rpy=0 0 0.0 -> xyz=0 0 0.165 rpy=0 0 0
