Commit message: kinsovler plugin calibration

File: src/gzrcs/config/FanucLRMate200iD.urdf (robot description, URDF)
Before this commit: robot fanuc_lrmate200id, 7 links, 6 joints
Links:
- link fanuc_base_link: mass 4 -> None

Commit message: yeat again update

File: src/gzrcs/config/FanucLRMate200iD.urdf (robot description, URDF)
Before this commit: robot fanuc_lrmate200id, 7 links, 6 joints
Links:
- link fanuc_base_link: mass None -> 4

File: src/gzrcs/config/lrmate200id.urdf (robot description, URDF)
Before this commit: robot fanuc_lrmate200id, 10 links, 9 joints
Joints:
- joint fanuc_joint_5: child fanuc_link_5 -> link_5; parent fanuc_link_4 -> link_4
